File: PCB/Project/Audio_Mixer/Audio_Mixer.kicad_sch (KiCad schematic)
At the start: 36 parts, among them J1 ASJ-195-L-HT, J2 SJ-435107RS, J3 ASJ-195-L-HT, J4 ASJ-195-L-HT, J5 ASJ-195-L-HT, J6 UJC-HP-3-SMT-TR, U1 MAX97220A

Commit message: Boards ordered for v0; gerbs included
Parts:
- removed RV1: L_Trim_50k, symbol Device:R_Potentiometer_Trim
- removed RV2: R_Trim_50k, symbol Device:R_Potentiometer_Trim
- added RV1: Trim_100k, patchez_audio:PS30-2, symbol Device:R_Potentiometer_Dual_Separate
- C12: value 1u -> 0.1u
- J1, J3, J4, J5: footprint (none) -> patchez_audio:ASJ-195-X-HT
- RV3: value Gain_50k -> Gain_100k; footprint (none) -> patchez_audio:RK14K124
- RV4, RV5: footprint (none) -> patchez_audio:RK14K124
Connections:
- net INR-: now also RV3.2; no longer RV3.1
- net Line0_L: now also RV4.6; no longer RV4.4
- net Line0_R: now also RV4.3; no longer RV4.1
- net Line0_SW: now also RV4.1, RV4.4; no longer RV4.3, RV4.6
- net Line1_L: now also RV5.6; no longer RV5.4
- net Line1_R: now also RV5.3; no longer RV5.1
- net Line1_SW: now also RV5.1, RV5.4; no longer RV5.3, RV5.6
- net OUTL: now also RV1.5
- net OUTR: now also RV3.1, RV1.2; no longer RV3.2
- net at R4.2: now also RV1.4
- net at R1.2: now also RV1.1
Other:
- moved on the sheet: RV3A
Changed lines of the file:
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@@
   (no_connect (at 144.78 80.01))
   (no_connect (at 151.13 88.9))
-  (no_connect (at 144.78 52.07))
+  (no_connect (at 140.97 55.88))
   (no_connect (at 151.13 60.96))
   (wire (pts (xy 231.14 48.26) (xy 232.41 48.26))
@@
         (path "/834077f0-32d5-4fe7-bf02-514f1118af40"
           (reference "R4") (unit 1)
-        )
-      )
-    )
-  )
-  (symbol (lib_id "Device:R_Potentiometer_Trim") (at 147.32 88.9 270) (mirror x) (unit 1)
-    (in_bom yes) (on_board yes) (dnp no)
-    (property "Reference" "RV1" (at 147.32 91.44 90)
-      (effects (font (size 1.27 1.27)))
-    )
-    (property "Value" "L_Trim_50k" (at 147.32 93.98 90)
-      (effects (font (size 1.27 1.27)))
-    )
-    (property "Footprint" "" (at 147.32 88.9 0)
-      (effects (font (size 1.27 1.27)) hide)
-    )
-    (property "Datasheet" "~" (at 147.32 88.9 0)
-      (effects (font (size 1.27 1.27)) hide)
-    )
-    (pin "1")
-    (pin "2")
-    (pin "3")
-    (instances
-      (project "Audio_Mixer"
-        (path "/834077f0-32d5-4fe7-bf02-514f1118af40"
-          (reference "RV1") (unit 1)
         )
       )
@@
     )
   )
-  (symbol (lib_id "Device:R_Potentiometer_Trim") (at 147.32 60.96 270) (mirror x) (unit 1)
-    (in_bom yes) (on_board yes) (dnp no)
-    (property "Reference" "RV2" (at 144.78 63.5 90)
-      (effects (font (size 1.27 1.27)))
-    )
-    (property "Value" "R_Trim_50k" (at 152.4 63.5 90)
-      (effects (font (size 1.27 1.27)))
-    )
-    (property "Footprint" "" (at 147.32 60.96 0)
+  (symbol (lib_id "Device:R_Potentiometer_Dual_Separate") (at 147.32 60.96 90) (unit 1)
+    (in_bom yes) (on_board yes) (dnp no)
+    (property "Reference" "RV1" (at 147.32 63.5 90)
+      (effects (font (size 1.27 1.27)))
+    )
+    (property "Value" "Trim_100k" (at 147.32 65.405 90)
+      (effects (font (size 1.27 1.27)))
+    )
+    (property "Footprint" "patchez_audio:PS30-2" (at 147.32 60.96 0)
       (effects (font (size 1.27 1.27)) hide)
     )
@@
     (pin "2")
     (pin "3")
-    (instances
-      (project "Audio_Mixer"
-        (path "/834077f0-32d5-4fe7-bf02-514f1118af40"
-          (reference "RV2") (unit 1)
+    (pin "4")
+    (pin "5")
+    (pin "6")
+    (instances
+      (project "Audio_Mixer"
+        (path "/834077f0-32d5-4fe7-bf02-514f1118af40"
+          (reference "RV1") (unit 1)
         )
       )
@@
       (effects (font (size 1.27 1.27)))
     )
-    (property "Value" "Gain_50k" (at 140.97 84.455 90)
-      (effects (font (size 1.27 1.27)))
-    )
-    (property "Footprint" "" (at 140.97 80.01 0)
+    (property "Value" "Gain_100k" (at 140.97 84.455 90)
+      (effects (font (size 1.27 1.27)))
+    )
+    (property "Footprint" "patchez_audio:RK14K124" (at 140.97 80.01 0)
       (effects (font (size 1.27 1.27)) hide)
     )
@@
       (effects (font (size 1.27 1.27)))
     )
-    (property "Footprint" "" (at 25.4 119.38 0)
+    (property "Footprint" "patchez_audio:ASJ-195-X-HT" (at 25.4 119.38 0)
       (effects (font (size 1.27 1.27)) hide)
     )
@@
       (effects (font (size 1.27 1.27)) (justify left))
     )
-    (property "Value" "1u" (at 66.675 167.005 0)
+    (property "Value" "0.1u" (at 66.675 167.005 0)
       (effects (font (size 1.27 1.27)) (justify left))
     )
@@
     )
   )
-  (symbol (lib_id "Device:R_Potentiometer_Dual_Separate") (at 142.24 123.19 0) (unit 1)
-    (in_bom yes) (on_board yes) (dnp no) (fields_autoplaced)
-    (property "Reference" "RV4" (at 139.7 121.92 0)
+  (symbol (lib_id "Device:R_Potentiometer_Dual_Separate") (at 142.24 123.19 0) (mirror x) (unit 1)
+    (in_bom yes) (on_board yes) (dnp no)
+    (property "Reference" "RV4" (at 139.7 124.46 0)
       (effects (font (size 1.27 1.27)) (justify right))
     )
-    (property "Value" "Line0_V" (at 139.7 124.46 0)
+    (property "Value" "Line0_V" (at 139.7 121.92 0)
       (effects (font (size 1.27 1.27)) (justify right))
     )
-    (property "Footprint" "" (at 142.24 123.19 0)
+    (property "Footprint" "patchez_audio:RK14K124" (at 142.24 123.19 0)
       (effects (font (size 1.27 1.27)) hide)
     )
@@
     )
   )
-  (symbol (lib_id "Device:R_Potentiometer_Dual_Separate") (at 142.24 140.97 0) (unit 1)
-    (in_bom yes) (on_board yes) (dnp no) (fields_autoplaced)
-    (property "Reference" "RV5" (at 139.7 139.7 0)
+  (symbol (lib_id "Device:R_Potentiometer_Dual_Separate") (at 142.24 140.97 0) (mirror x) (unit 1)
+    (in_bom yes) (on_board yes) (dnp no)
+    (property "Reference" "RV5" (at 139.7 142.24 0)
       (effects (font (size 1.27 1.27)) (justify right))
     )
-    (property "Value" "Line1_V" (at 139.7 142.24 0)
+    (property "Value" "Line1_V" (at 139.7 139.7 0)
       (effects (font (size 1.27 1.27)) (justify right))
     )
-    (property "Footprint" "" (at 142.24 140.97 0)
+    (property "Footprint" "patchez_audio:RK14K124" (at 142.24 140.97 0)
       (effects (font (size 1.27 1.27)) hide)
     )
@@
       (effects (font (size 1.27 1.27)))
     )
-    (property "Footprint" "" (at 73.66 119.38 0)
+    (property "Footprint" "patchez_audio:ASJ-195-X-HT" (at 73.66 119.38 0)
       (effects (font (size 1.27 1.27)) hide)
     )
@@
       (effects (font (size 1.27 1.27)))
     )
-    (property "Footprint" "" (at 25.4 58.42 0)
+    (property "Footprint" "patchez_audio:ASJ-195-X-HT" (at 25.4 58.42 0)
       (effects (font (size 1.27 1.27)) hide)
     )
@@
     )
   )
-  (symbol (lib_id "Device:R_Potentiometer_Dual_Separate") (at 109.22 123.19 0) (unit 2)
-    (in_bom yes) (on_board yes) (dnp no) (fields_autoplaced)
-    (property "Reference" "RV4" (at 106.68 121.92 0)
+  (symbol (lib_id "Device:R_Potentiometer_Dual_Separate") (at 109.22 123.19 0) (mirror x) (unit 2)
+    (in_bom yes) (on_board yes) (dnp no)
+    (property "Reference" "RV4" (at 106.68 124.46 0)
       (effects (font (size 1.27 1.27)) (justify right))
     )
-    (property "Value" "Line0_V" (at 106.68 124.46 0)
+    (property "Value" "Line0_V" (at 106.68 121.92 0)
       (effects (font (size 1.27 1.27)) (justify right))
     )
-    (property "Footprint" "" (at 109.22 123.19 0)
+    (property "Footprint" "patchez_audio:RK14K124" (at 109.22 123.19 0)
       (effects (font (size 1.27 1.27)) hide)
     )
@@
     )
   )
-  (symbol (lib_id "Device:R_Potentiometer_Dual_Separate") (at 109.22 140.97 0) (unit 2)
-    (in_bom yes) (on_board yes) (dnp no) (fields_autoplaced)
-    (property "Reference" "RV5" (at 106.68 139.7 0)
+  (symbol (lib_id "Device:R_Potentiometer_Dual_Separate") (at 109.22 140.97 0) (mirror x) (unit 2)
+    (in_bom yes) (on_board yes) (dnp no)
+    (property "Reference" "RV5" (at 106.68 142.24 0)
       (effects (font (size 1.27 1.27)) (justify right))
     )
-    (property "Value" "Line1_V" (at 106.68 142.24 0)
+    (property "Value" "Line1_V" (at 106.68 139.7 0)
       (effects (font (size 1.27 1.27)) (justify right))
     )
-    (property "Footprint" "" (at 109.22 140.97 0)
+    (property "Footprint" "patchez_audio:RK14K124" (at 109.22 140.97 0)
       (effects (font (size 1.27 1.27)) hide)
     )
@@
     )
   )
-  (symbol (lib_id "Device:R_Potentiometer_Dual_Separate") (at 140.97 52.07 90) (unit 1)
-    (in_bom yes) (on_board yes) (dnp no)
-    (property "Reference" "RV3" (at 140.97 54.61 90)
-      (effects (font (size 1.27 1.27)))
-    )
-    (property "Value" "Gain_50k" (at 140.97 56.515 90)
-      (effects (font (size 1.27 1.27)))
-    )
-    (property "Footprint" "" (at 140.97 52.07 0)
+  (symbol (lib_id "Device:R_Potentiometer_Dual_Separate") (at 140.97 52.07 0) (mirror y) (unit 1)
+    (in_bom yes) (on_board yes) (dnp no)
+    (property "Reference" "RV3" (at 143.51 52.07 90)
+      (effects (font (size 1.27 1.27)))
+    )
+    (property "Value" "Gain_100k" (at 145.415 52.07 90)
+      (effects (font (size 1.27 1.27)))
+    )
+    (property "Footprint" "patchez_audio:RK14K124" (at 140.97 52.07 0)
       (effects (font (size 1.27 1.27)) hide)
     )
@@
       (effects (font (size 1.27 1.27)))
     )
-    (property "Footprint" "" (at 25.4 88.9 0)
+    (property "Footprint" "patchez_audio:ASJ-195-X-HT" (at 25.4 88.9 0)
       (effects (font (size 1.27 1.27)) hide)
     )
@@
         )
       )
+    )
+  )
+  (symbol (lib_id "Device:R_Potentiometer_Dual_Separate") (at 147.32 88.9 90) (unit 2)
+    (in_bom yes) (on_board yes) (dnp no)
+    (property "Reference" "RV1" (at 147.32 91.44 90)
+      (effects (font (size 1.27 1.27)))
+    )
+    (property "Value" "Trim_100k" (at 147.32 93.345 90)
+      (effects (font (size 1.27 1.27)))
+    )
+    (property "Footprint" "patchez_audio:PS30-2" (at 147.32 88.9 0)
+      (effects (font (size 1.27 1.27)) hide)
+    )
+    (property "Datasheet" "~" (at 147.32 88.9 0)
+      (effects (font (size 1.27 1.27)) hide)
+    )
+    (pin "1")
+    (pin "2")
+    (pin "3")
+    (pin "4")
+    (pin "5")
+    (pin "6")
+    (instances
+      (project "Audio_Mixer"
+        (path "/834077f0-32d5-4fe7-bf02-514f1118af40"
+          (reference "RV1") (unit 2)
+        )
+      )
